File: Hardware/RotatingSignalStack_board/_autosave-RotatingSignalStack_board.kicad_pcb (KiCad board)
At the start: 2 copper layers, 39 parts, among them J2 RJ45_LED_Shielded, Q9 Q_PMOS_DGS, SW1 SW_Push, SW2 SW_Push, U1 OKI, U2 SMAJ12CA, U3 Teensy4.1_DEV-16771, U4 TSR_1-2450, U5 LSM303C

Commit message: file cleanup
Parts:
- removed J2: RJ45_LED_Shielded, MRDT_Connectors:RJ45_Teensy
- removed U2: SMAJ12CA, MRDT_Actives:DO-214AC
- added Conn2: AndersonPP, MRDT_Connectors:Square_Anderson_2_H_Side_By_Side, F.Cu at (66.0, 26.7)
- added Conn4: AndersonPP, MRDT_Connectors:Square_Anderson_2_H_Side_By_Side, F.Cu at (66.0, 43.6)
- added Conn5: Molex_SL_02, MRDT_Connectors:MOLEX_SL_02_Horizontal, F.Cu at (71.3, 36.5)
- added D4: B120-E3, Diode_SMD:D_SMA, F.Cu at (71.7, 40.6)
Connections:
- C10 pad 1: +3V3 -> +3.3V
- C2 pad 1: +3V3 -> +3.3V
- C3 pad 1: Net-(Conn1B-V+Log) -> Net-(Conn3B-V+Log)
- C4 pad 1: Net-(Conn1B-V+Log) -> Net-(Conn3B-V+Log)
- C5 pad 1: Net-(Conn1B-V+Log) -> Net-(Conn3B-V+Log)
- C8 pad 1: +3V3 -> +3.3V
- C9 pad 1: +3V3 -> +3.3V
- Conn1 pad 2: Net-(Conn1B-V+Log) -> (no net)
- Conn3 pad 1: GND -> (no net)
- Conn3 pad 2: Net-(Conn1B-V+Log) -> Net-(Conn3B-V+Log)
- Q9 pad 2: Net-(Conn1B-V+Log) -> Net-(Conn3B-V+Log)
- R1 pad 1: +3V3 -> +3.3V
- R4 pad 1: +3V3 -> +3.3V
- R5 pad 1: +3V3 -> +3.3V
- SW1 pad 1: +3V3 -> +3.3V
- SW2 pad 1: +3V3 -> +3.3V
- U1 pad 3: +3V3 -> +3.3V
- U5 pad 10: +3V3 -> +3.3V
- U5 pad 7: MAG INT DATA READY -> unconnected-(U5-INT_MAG-Pad7)
- U5 pad 9: +3V3 -> +3.3V
