File: RotatingSignalStack/oscillator.kicad_sch (KiCad schematic)
At the start: 3 parts, among them U5 SG-210STF 50.0000ML0

Commit message: Added everything
Parts:
- R14, R5: footprint (none) -> Resistor_SMD:R_0603_1608Metric_Pad0.98x0.95mm_HandSolder
- U5: footprint SG-210STF 50.0000ML0_EPS -> SignalStack:SG-210STF 50.0000ML0_EPS
Changed lines of the file:
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@@
 			)
 		)
-		(property "Footprint" ""
+		(property "Footprint" "Resistor_SMD:R_0603_1608Metric_Pad0.98x0.95mm_HandSolder"
 			(at 223.774 106.934 90)
 			(effects
@@
 			)
 		)
-		(property "Footprint" ""
+		(property "Footprint" "Resistor_SMD:R_0603_1608Metric_Pad0.98x0.95mm_HandSolder"
 			(at 223.774 96.774 90)
 			(effects
@@
 			)
 		)
-		(property "Footprint" "SG-210STF 50.0000ML0_EPS"
+		(property "Footprint" "SignalStack:SG-210STF 50.0000ML0_EPS"
 			(at 106.68 100.33 0)
 			(effects
