File: RotatingSignalStack/stm.kicad_sch (KiCad schematic)
At the start: 16 parts, among them IC2 STM32H562RIT6, SW1 SW_Push, SW2 Boot Switch

Commit message: placement fix
Parts:
- removed C21: 100nF, Capacitor_SMD:C_0603_1608Metric_Pad1.08x0.95mm_HandSolder, symbol Device:C
- added C4: 2.2uF, Capacitor_SMD:C_0603_1608Metric_Pad1.08x0.95mm_HandSolder, symbol Device:C
- added J1: Conn_ARM_SWD_TagConnect_TC2030-NL, Connector:Tag-Connect_TC2030-IDC-NL_2x03_P1.27mm_Vertical, symbol Connector:Conn_ARM_SWD_TagConnect_TC2030-NL
- C12, C13, C19, C20, C31, C35: value 100nF -> 0.1uF
- C30: value 4.7nF -> 4.7uF
- C33: value 2.2uF -> 0.1uF
Connections:
- net +3V3: now also C19.1, C20.1, C33.1, J1.1 (VCC)
- net GND: now also C13.2, C19.2, C20.2, C32.1, C33.2, C4.1, J1.5 (GND); no longer C33.1
- net NRST: now also J1.3 (~{RESET})
- net SWDIO: now also J1.2 (SWDIO)
- net SWO: now also J1.6 (SWO)
- net VCAP1: now also C4.2
- new net SWDCLK: J1.4 (SWCLK)
Other:
- moved on the sheet: C30, C31, C32, C34, C35

Commit message: layout
Parts:
- removed J1: Conn_ARM_SWD_TagConnect_TC2030-NL, Connector:Tag-Connect_TC2030-IDC-NL_2x03_P1.27mm_Vertical, symbol Connector:Conn_ARM_SWD_TagConnect_TC2030-NL
- added J2: Conn_01x04, Connector_PinSocket_2.54mm:PinSocket_1x04_P2.54mm_Vertical, symbol Connector_Generic:Conn_01x04
Connections:
- net SWCLK is gone; now on net SWDCLK: IC2.49 (PA14)
- net +3V3: now also J2.1 (Pin_1)
- net GND: now also J2.4 (Pin_4)
- net SWDCLK: now also J2.2 (Pin_2)
- net SWDIO: now also J2.3 (Pin_3)
- net NRST: no longer names the net of C12.1, D7.1, IC2.7 (NRST), SW1.1
- net SWO: no longer names the net of IC2.55 (PB3)
- no-connect marks 28 -> 29

Commit message: new one
Connections:
- net ALIGN: now also IC2.6 (PH1-OSC_OUT); no longer IC2.51 (PC10)
- net JOG A: now also IC2.3 (PC14-OSC32_IN); no longer IC2.53 (PC12)
- net JOG B: now also IC2.4 (PC15-OSC32_OUT); no longer IC2.52 (PC11)
- no-connect marks 29 -> 26
Other:
- note removed: "GPIO->"
Changed lines of the file:
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@@
 	(generator_version "9.0")
 	(paper "A4")
-	(text "GPIO->"
-		(exclude_from_sim no)
-		(at 80.518 101.854 0)
-		(effects
-			(font
-				(size 1.27 1.27)
-			)
-		)
-	)
 	(text "USED DIFFERENT CHIP EXAMPLE (couldn't find one for this exact chip):\nhttps://www.st.com/resource/en/schematic_pack/mb1404-h563zi-c01-schematic.pdf"
 		(exclude_from_sim no)
@@
 	)
 	(no_connect
-		(at 86.36 101.6)
-	)
-	(no_connect
 		(at 139.7 111.76)
 	)
@@
 	)
 	(no_connect
-		(at 86.36 96.52)
-	)
-	(no_connect
 		(at 129.54 71.12)
-	)
-	(no_connect
-		(at 86.36 93.98)
 	)
 	(no_connect
@@
 		)
 	)
-	(hierarchical_label "JOG B"
+	(hierarchical_label "ALIGN"
 		(shape input)
-		(at 124.46 71.12 90)
-		(effects
-			(font
-				(size 1.27 1.27)
-			)
-			(justify left)
-		)
-	)
-	(hierarchical_label "JOG A"
-		(shape input)
-		(at 121.92 71.12 90)
-		(effects
-			(font
-				(size 1.27 1.27)
-			)
-			(justify left)
+		(at 86.36 101.6 180)
+		(effects
+			(font
+				(size 1.27 1.27)
+			)
+			(justify right)
 		)
 	)
@@
 		)
 	)
+	(hierarchical_label "JOG A"
+		(shape input)
+		(at 86.36 93.98 180)
+		(effects
+			(font
+				(size 1.27 1.27)
+			)
+			(justify right)
+		)
+	)
 	(hierarchical_label "MDIO"
 		(shape bidirectional)
@@
 		)
 	)
-	(hierarchical_label "ALIGN"
+	(hierarchical_label "JOG B"
 		(shape input)
-		(at 127 71.12 90)
-		(effects
-			(font
-				(size 1.27 1.27)
-			)
-			(justify left)
-		)
-	)
+		(at 86.36 96.52 180)
+		(effects
+			(font
+				(size 1.27 1.27)
+			)
+			(justify right)
+		)
+	)
