File: RotatingSignalStack/RotatingSignalStack.kicad_pcb (KiCad board)
At the start: 2 copper layers, 102.1 x 56.4 mm, 92 parts, among them IC2 STM32H562RIT6, J2 Conn_01x04, J3 RJ45_LED_Shielded, SW1 SW_Push, SW2 Boot Switch, SW5 SW_Push, SW6 SW_Push, SW7 SW_Push, T1 GMG116S1202R, U1 TMAG5273C1QDBVR, U2 AP63203WU-7, U3 SN65HVD232, U4 DP83825I, U5 SG-210STF 50.0000ML0, U6 USBLC6-2SC6, U7 USBLC6-4SC6

Commit message: layout
Parts:
- moved R11 23.7 mm to (155.2, 85.2)
- moved R7 16.5 mm to (155.2, 87.0)
- moved C30 9.67 mm to (171.8, 58.3), turned to -45 degrees
- moved C4 9.55 mm to (158.1, 63.4), turned to -135 degrees
- moved R15 8.64 mm to (164.0, 60.1), turned to 45 degrees
- moved C19 8.49 mm to (170.6, 59.6), turned to -45 degrees
- moved C20 8.20 mm to (159.4, 64.6), turned to 45 degrees
- moved C31 7.49 mm to (158.6, 70.0), turned to 135 degrees
- moved D7 6.66 mm to (173.4, 77.6), turned to 45 degrees
- moved C32 6.62 mm to (176.9, 72.0), turned to 45 degrees
- moved C35 6.44 mm to (161.9, 75.8), turned to 135 degrees
- moved C12 5.58 mm to (172.3, 76.6), turned to 45 degrees
- moved C13 5.55 mm to (175.6, 70.7), turned to -135 degrees
- moved C6 5.16 mm to (136.3, 92.5)
- moved C7 5.09 mm to (136.3, 90.7)
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Connections:
- net Net-(U4-RD+) renamed Rx+
- net Net-(U4-RD-) renamed Rx-
- net Net-(U4-TD+) renamed Tx+
- net Net-(U4-TD-) renamed Tx-
Routing:
- net VBAT: track 0.00 -> 65.2 mm, vias 0 -> 2
- net VBUS: track 0.00 -> 51.0 mm
- net VSSA: track 0.00 -> 41.4 mm
- net /Ethernet and Magnetics/Tx+: track 0.00 -> 36.8 mm, vias 0 -> 2
- net /Ethernet and Magnetics/Rx-: track 0.00 -> 36.7 mm, vias 0 -> 2
- net /Ethernet and Magnetics/Tx-: track 0.00 -> 36.7 mm, vias 0 -> 2
- net /Ethernet and Magnetics/Rx+: track 0.00 -> 36.6 mm, vias 0 -> 2
- net /PHY/TX_D0: track 0.00 -> 35.7 mm, vias 0 -> 2
- net /PHY/TX_D1: track 0.00 -> 35.6 mm, vias 0 -> 2
- net Net-(U7-VBUS): track 0.00 -> 32.2 mm
- net Net-(J3-Pad6): track 0.00 -> 27.5 mm
- net /PHY/TX_EN: track 0.00 -> 25.6 mm
- net /PHY/RST: track 0.00 -> 25.2 mm
- net Net-(C9-Pad1): track 0.00 -> 21.3 mm, vias 0 -> 2
- net Net-(J3-Pad3): track 0.00 -> 20.6 mm
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- added copper zone on B.Cu, net VSSA
- added copper zone on F.Cu, net VSSA
- removed copper zone on B.Cu, net GNDPWR

Commit message: more layout
Parts:
- C1, C10, C11, C12, C13, C14, C15, C16, C17, C18, C19, C2, C20, C22, C23, C24, C25, C26, C27, C28, C29, C3, C30, C31, C32, C33, C34, C35, C37, C4, C5, C7, C8, C9: footprint Capacitor_SMD:C_0603_1608Metric_Pad1.08x0.95mm_HandSolder -> Capacitor_SMD:C_0402_1005Metric_Pad0.74x0.62mm_HandSolder
- Conn1: footprint MRDT_Connectors:MOLEX_SL_04_Horizontal -> MRDT_Connectors:MOLEX_SL_04_Vertical
- R23: value 2.2k -> 1.5k
- moved R9 59.8 mm to (148.1, 105.4), turned to 90 degrees
- moved Conn1 58.0 mm to (140.7, 99.1)
- moved CR1 55.7 mm to (150.9, 105.4), turned to 180 degrees
- moved U3 48.1 mm to (156.7, 105.4), turned to 180 degrees
- moved R11 39.9 mm to (119.9, 103.9)
- moved R7 36.0 mm to (119.9, 80.0)
- moved C32 18.9 mm to (160.0, 63.5), turned to -45 degrees
- moved C4 18.8 mm to (174.8, 72.1), turned to 135 degrees
- moved R12 6.22 mm to (172.2, 83.6), turned to -90 degrees
- moved D7 5.06 mm to (176.5, 73.7)
- moved J3 4.85 mm to (109.7, 91.7), turned to -90 degrees
- moved R2 4.77 mm to (123.7, 83.3)
- moved C12 4.10 mm to (176.3, 75.4), turned to -135 degrees
- moved C9 4.10 mm to (125.5, 100.1), turned to 0 degrees
- moved R1 3.99 mm to (123.4, 99.3)
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Connections:
- net Net-(J3-Pad1) renamed /Ethernet and Magnetics/Txx+
- net Net-(J3-Pad2) renamed /Ethernet and Magnetics/Txx-
- net Net-(J3-Pad3) renamed /Ethernet and Magnetics/Rxx+
- net Net-(J3-Pad6) renamed /Ethernet and Magnetics/Rxx-
- net Rx+ renamed Net-(U4-RD+)
- net Rx- renamed Net-(U4-RD-)
- net Tx+ renamed Net-(U4-TD+)
- net Tx- renamed Net-(U4-TD-)
- C13 pad 1: VBAT -> VDD1
- C14 pad 1: VBAT -> VDD1
- C19 pad 1: VBAT -> VDD1
- C20 pad 1: VBAT -> VDD1
- C3 pad 1: VBAT -> VDD1
- C30 pad 1: VBAT -> VDD1
- C31 pad 1: VBAT -> VDD1
- C32 pad 2: VCAP1 -> VCAP2
- C33 pad 1: VBAT -> VDD1
- C34 pad 1: VBAT -> VDD1
- C35 pad 1: VBAT -> VDD1
- C37 pad 1: VBAT -> VDD1
- D1 pad 2: VBAT -> VDD1
- FB1 pad 2: VBAT -> VDD1
- FB2 pad 1: VBAT -> VDD1
- FB4 pad 2: VBAT -> VDD1
- IC2 pad 13: VBAT -> VDD1
- IC2 pad 19: VBAT -> VDD1
- IC2 pad 32: VBAT -> VDD1
- IC2 pad 48: VBAT -> VDD1
- IC2 pad 62: VCAP1 -> VCAP2
- IC2 pad 64: VBAT -> VDD1
- J2 pad 1: VBAT -> VDD1
- L1 pad 2: VBAT -> VDD1
- R10 pad 1: VBAT -> VDD1
- R6 pad 1: VBAT -> VDD1
- SW2 pad 3: VBAT -> VDD1
- U1 pad 4: VBAT -> VDD1
- U2 pad 1: VBAT -> VDD1
- U3 pad 3: VBAT -> VDD1
- U4 pad 3: VBAT -> VDD1
- U5 pad 1: VBAT -> VDD1
- U5 pad 4: VBAT -> VDD1
Routing:
- net VBAT: track 65.2 -> 0.00 mm, vias 2 -> 0
- net VBUS: track 51.0 -> 0.00 mm
- net VDD1: track 0.00 -> 47.9 mm, vias 0 -> 2
- net VSSA: track 41.4 -> 14.6 mm
- net /PHY/RX_D1: track 0.00 -> 20.2 mm
- net /PHY/RX_D0: track 0.00 -> 18.9 mm
- net /Ethernet and Magnetics/Rxx-: track 27.5 -> 13.0 mm
- net /CAN/CANL: track 0.00 -> 13.8 mm
- net /CAN/CANH: track 0.00 -> 13.8 mm
- net /Ethernet and Magnetics/LED2: track 0.00 -> 9.93 mm
- net /Ethernet and Magnetics/LED0: track 0.00 -> 7.88 mm
- net Net-(U4-VDDIO): track 4.25 -> 10.4 mm, vias 0 -> 2
- net /Ethernet and Magnetics/Rxx+: track 20.6 -> 14.6 mm
- net /Ethernet and Magnetics/Txx-: track 17.7 -> 12.3 mm
- net Net-(U2-SW): track 4.92 -> 0.00 mm
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- added copper zone on B.Cu, net GNDPWR

Commit message: layout 3
Parts:
- C36, C6: footprint Capacitor_SMD:C_0603_1608Metric_Pad1.08x0.95mm_HandSolder -> Capacitor_SMD:C_0402_1005Metric_Pad0.74x0.62mm_HandSolder
- moved SW2 91.3 mm to (208.2, 32.0)
- moved H2 77.0 mm to (189.0, 64.0)
- moved H3 66.8 mm to (131.2, 102.5), turned to 180 degrees
- moved R10 65.9 mm to (237.0, 31.1)
- moved R6 65.9 mm to (230.9, 31.1)
- moved C14 65.9 mm to (237.3, 35.2)
- moved U1 65.9 mm to (233.9, 35.1)
- moved U6 65.9 mm to (234.0, 31.4)
- moved R18 55.6 mm to (177.4, 35.0)
- moved SW5 55.6 mm to (174.5, 31.5)
- moved D10 55.6 mm to (161.5, 35.0)
- moved D3 55.6 mm to (171.5, 35.0)
- moved SW7 55.6 mm to (164.3, 31.5)
- moved D9 55.6 mm to (181.8, 35.0)
- moved R17 55.6 mm to (187.4, 35.0)
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Connections:
- C13 pad 1: VDD1 -> VBAT
- C14 pad 1: VDD1 -> VBAT
- C19 pad 1: VDD1 -> VBAT
- C20 pad 1: VDD1 -> VBAT
- C3 pad 1: VDD1 -> VBAT
- C30 pad 1: VDD1 -> VBAT
- C31 pad 1: VDD1 -> VBAT
- C33 pad 1: VDD1 -> VBAT
- C34 pad 1: VDD1 -> VBAT
- C35 pad 1: VDD1 -> VBAT
- C37 pad 1: VDD1 -> VBAT
- D1 pad 2: VDD1 -> VBAT
- FB1 pad 2: VDD1 -> VBAT
- FB2 pad 1: VDD1 -> VBAT
- FB4 pad 2: VDD1 -> VBAT
- IC2 pad 13: VDD1 -> VBAT
- IC2 pad 19: VDD1 -> VBAT
- IC2 pad 32: VDD1 -> VBAT
- IC2 pad 48: VDD1 -> VBAT
- IC2 pad 64: VDD1 -> VBAT
- J2 pad 1: VDD1 -> VBAT
- L1 pad 2: VDD1 -> VBAT
- R10 pad 1: VDD1 -> VBAT
- R6 pad 1: VDD1 -> VBAT
- SW2 pad 3: VDD1 -> VBAT
- U1 pad 4: VDD1 -> VBAT
- U2 pad 1: VDD1 -> VBAT
- U3 pad 3: VDD1 -> VBAT
- U4 pad 3: VDD1 -> VBAT
- U5 pad 1: VDD1 -> VBAT
- U5 pad 4: VDD1 -> VBAT
Routing:
- net VDD1: track 47.9 -> 0.00 mm, vias 2 -> 0
- net VBAT: track 0.00 -> 37.7 mm, vias 0 -> 1
- net Net-(C9-Pad1): track 19.6 -> 0.00 mm
- net /Ethernet and Magnetics/Rx-: track 36.7 -> 18.9 mm
- net /Ethernet and Magnetics/Tx-: track 36.7 -> 19.1 mm
- net /Ethernet and Magnetics/Tx+: track 36.8 -> 19.2 mm
- net /Ethernet and Magnetics/Rx+: track 36.6 -> 19.0 mm
- net VSSA: track 14.6 -> 0.00 mm, vias 0 -> 1
- net /CAN/CANL: track 13.8 -> 0.00 mm
- net /CAN/CANH: track 13.8 -> 0.00 mm
- net Net-(U4-50MHzOut/LED2/S(RX_DV_EN)): track 15.7 -> 5.49 mm, vias 2 -> 0
- net Net-(C5-Pad1): track 8.30 -> 0.00 mm, vias 2 -> 0
- net Net-(C7-Pad1): track 8.19 -> 0.00 mm, vias 3 -> 0
- net Net-(U4-LED0/S(ANEG_Dis)): track 14.8 -> 8.18 mm, vias 2 -> 0
- net Net-(R2-Pad1): track 6.16 -> 0.00 mm
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- removed copper zone on B.Cu, net GNDPWR
- removed copper zone on F.Cu, net GNDPWR
- removed copper zone on B.Cu, net VSSA
- removed copper zone on F.Cu, net VSSA
Other:
- board outline removed
