File: RotatingSignalStack/_autosave-stm.kicad_sch (KiCad schematic)
At the start: 20 parts, among them IC2 STM32H562RIT6, J1 Conn_01x06, J2 Conn_01x04, J4 Conn_01x09, SW1 SW_Push, U8 OKI-78SR-3.3_1.5-W36-C

Commit message: final layout
Parts:
- C12: footprint Capacitor_SMD:C_0402_1005Metric_Pad0.74x0.62mm_HandSolder -> Capacitor_SMD:C_0603_1608Metric_Pad1.08x0.95mm_HandSolder
Changed lines of the file:
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@@
 			)
 		)
-		(property "Footprint" "Capacitor_SMD:C_0402_1005Metric_Pad0.74x0.62mm_HandSolder"
+		(property "Footprint" "Capacitor_SMD:C_0603_1608Metric_Pad1.08x0.95mm_HandSolder"
 			(at 25.0952 116.84 0)
 			(effects
