File: board/rotating_signal_stack.kicad_sch (KiCad schematic)
At the start: 25 parts, among them J1 RJ45_LED_Shielded, J3 Motor pins, J4 Molex_Megafit_02, Q1 TPC8132_LQS, SW1 SW_Push, SW2 SW_Push

Commit message: Made some progress in the footprint.
I need to change the STM32CubeMX pin locations to make the footprint less messy, but I will work on this more sometime next week.
Parts:
- added U4: (no value), Connector_PinHeader_2.54mm:PinHeader_1x05_P2.54mm_Vertical, symbol RotatingSignalStack_Symbols:Adafruit_QMC5883P
- C3: value 0.1 uF -> 10 uF
- J3: footprint Connector:NS-Tech_Grove_1x04_P2mm_Vertical -> MRDT_Connectors:MOLEX_SL_04_Horizontal
- SW1, SW2: footprint Button_Switch_THT:SW_NKK_GW12LJP -> MRDT_Switches:SW_SPST_TL3305A
Connections:
- net +3V3: now also U4.1 (VIN)
- net DIR: now also U2.28 (PB6); no longer U2.10 (PA10)
- net GND: now also U4.3 (GND)
- net M0: now also U1.2 (M0); no longer U1.4 (M2)
- net M2: now also U1.4 (M2); no longer U1.2 (M0)
- net SCL: now also U4.4 (SCL)
- net SDA: now also U4.5 (SDA)
- net nSTBY: now also U2.27 (PB5); no longer U2.18 (PB13)
- net at J3.1 (Pin_1): now also U1.11 (OUTB1); no longer U1.14 (OUTA1)
- net at J3.2 (Pin_2): now also U1.12 (OUTB2); no longer U1.13 (OUTA2)
- net at J3.3 (Pin_3): now also U1.13 (OUTA2); no longer U1.12 (OUTB2)
- net at J3.4 (Pin_4): now also U1.14 (OUTA1); no longer U1.11 (OUTB1)
- net INT: no longer names the net of U2.12 (PA8)
- no-connect marks 26 -> 28
Other:
- note added: "Magnometer"
- moved on the sheet: J3
